File: Tarea_2.kicad_pcb (KiCad board)
At the start: 2 copper layers, 11 parts, among them J1 54-00166, J2 PPTC241LFBN-RC, J3 PPTC241LFBN-RC, U2 TPS75318QPWPRQ1, U3 MIMXRT685SFVKB

Commit message: Version 1.0
Diseño inicial de la placa.
Parts:
- moved J1 55.1 mm to (132.5, 29.5)
- moved U3 48.4 mm to (152.0, 36.5)
- moved J3 45.9 mm to (159.5, 86.1), turned to 90 degrees
- moved U2 45.8 mm to (142.5, 40.0), turned to 90 degrees
- moved R2 36.4 mm to (149.7, 47.0)
- moved R1 36.3 mm to (149.8, 45.5)
- moved R3 36.1 mm to (149.7, 49.0)
- moved C2 31.5 mm to (148.0, 47.0)
- moved C1 31.4 mm to (148.0, 45.5)
- moved C3 31.2 mm to (148.0, 49.0)
- moved J2 28.2 mm to (125.0, 87.9), turned to 90 degrees

Commit message: Version 1.1
- Configuradas las 4 capas de la PCB
Routing:
- added copper zone on In2.Cu, net /Alimentacion/V18
- added copper zone on In1.Cu, net GND
Other:
- copper layers 2 -> 4
Changed lines of the file:
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@@
 	(layers
 		(0 "F.Cu" signal)
+		(4 "In1.Cu" signal)
+		(6 "In2.Cu" signal)
 		(2 "B.Cu" signal)
 		(9 "F.Adhes" user "F.Adhesive")
@@
 	)
 	(setup
+		(stackup
+			(layer "F.SilkS"
+				(type "Top Silk Screen")
+			)
+			(layer "F.Paste"
+				(type "Top Solder Paste")
+			)
+			(layer "F.Mask"
+				(type "Top Solder Mask")
+				(thickness 0.01)
+			)
+			(layer "F.Cu"
+				(type "copper")
+				(thickness 0.035)
+			)
+			(layer "dielectric 1"
+				(type "prepreg")
+				(thickness 0.1)
+				(material "FR4")
+				(epsilon_r 4.5)
+				(loss_tangent 0.02)
+			)
+			(layer "In1.Cu"
+				(type "copper")
+				(thickness 0.035)
+			)
+			(layer "dielectric 2"
+				(type "core")
+				(thickness 1.24)
+				(material "FR4")
+				(epsilon_r 4.5)
+				(loss_tangent 0.02)
+			)
+			(layer "In2.Cu"
+				(type "copper")
+				(thickness 0.035)
+			)
+			(layer "dielectric 3"
+				(type "prepreg")
+				(thickness 0.1)
+				(material "FR4")
+				(epsilon_r 4.5)
+				(loss_tangent 0.02)
+			)
+			(layer "B.Cu"
+				(type "copper")
+				(thickness 0.035)
+			)
+			(layer "B.Mask"
+				(type "Bottom Solder Mask")
+				(thickness 0.01)
+			)
+			(layer "B.Paste"
+				(type "Bottom Solder Paste")
+			)
+			(layer "B.SilkS"
+				(type "Bottom Silk Screen")
+			)
+			(copper_finish "None")
+			(dielectric_constraints no)
+		)
 		(pad_to_mask_clearance 0)
 		(allow_soldermask_bridges_in_footprints no)
@@
 		(capping no)
 		(filling no)
+		(zone_defaults)
 		(pcbplotparams
 			(layerselection 0x00000000_00000000_55555555_5755f5ff)
@@
 		(embedded_fonts no)
 	)
+	(gr_line
+		(start 119.5 24.5)
+		(end 119.5 93)
+		(stroke
+			(width 0.2)
+			(type default)
+		)
+		(layer "In2.Cu")
+	)
+	(gr_line
+		(start 119.5 24.5)
+		(end 166.5 24.5)
+		(stroke
+			(width 0.2)
+			(type default)
+		)
+		(layer "In2.Cu")
+	)
+	(gr_line
+		(start 166.5 24.5)
+		(end 166.5 93)
+		(stroke
+			(width 0.2)
+			(type default)
+		)
+		(layer "In2.Cu")
+	)
+	(gr_line
+		(start 166.5 93)
+		(end 119.5 93)
+		(stroke
+			(width 0.2)
+			(type default)
+		)
+		(layer "In2.Cu")
+	)
+	(zone
+		(net "GND")
+		(layer "In1.Cu")
+		(name "GND")
+		(hatch edge 0.5)
+		(connect_pads
+			(clearance 0.5)
+		)
+		(min_thickness 0.25)
+		(fill yes
+			(thermal_gap 0.5)
+			(thermal_bridge_width 0.5)
+			(island_removal_mode 0)
+		)
+		(polygon
+			(pts
+				(xy 116.5 23.5) (xy 168.5 23) (xy 168.5 95.5) (xy 116.5 96)
+			)
+		)
+	)
+	(zone
+		(net "/Alimentacion/V18")
+		(layer "In2.Cu")
+		(name "PWR_1")
+		(hatch edge 0.5)
+		(priority 1)
+		(connect_pads
+			(clearance 0.5)
+		)
+		(min_thickness 0.25)
+		(fill yes
+			(thermal_gap 0.5)
+			(thermal_bridge_width 0.5)
+			(island_removal_mode 0)
+		)
+		(polygon
+			(pts
+				(xy 119.5 24.5) (xy 166.5 24.5) (xy 166.5 93) (xy 119.5 93)
+			)
+		)
+	)
 	(embedded_fonts no)

Commit message: - Primer commit de la rama
Parts:
- removed J2: PPTC241LFBN-RC, Snapeda:CONN24_PPTC241LFBN-RC_SUL
- added C7: 4.7u, Capacitor_SMD:C_01005_0402Metric, F.Cu at (176.6, 46.9)
- moved J1 56.0 mm to (180.9, 57.5)
- moved U2 52.8 mm to (191.9, 58.7), turned to 0 degrees
- moved J3 50.9 mm to (178.9, 39.0), turned to 0 degrees
- moved C3 28.9 mm to (176.6, 45.3)
- moved C1 28.8 mm to (176.6, 42.0)
- moved C2 28.8 mm to (176.6, 43.6)
- moved R2 27.1 mm to (176.6, 50.2)
- moved R3 27.1 mm to (176.6, 51.9)
- moved R1 27.0 mm to (176.6, 48.6)
- moved U3 9.71 mm to (144.0, 42.0)
Connections:
- C2 pad 1: Net-(U3B-PIO2_26) -> Net-(U3B-PIO2_25)
- C3 pad 1: Net-(U3B-PIO2_28) -> Net-(U3B-PIO2_26)
- J3 pad 2: Net-(J3-Pad2) -> unconnected-(J3-Pad2)
- J3 pad 22: unconnected-(J3-Pad22) -> Net-(J3-Pad22)
- J3 pad 23: unconnected-(J3-Pad23) -> Net-(J3-Pad23)
- J3 pad 24: unconnected-(J3-Pad24) -> Net-(J3-Pad24)
- J3 pad 4: Net-(J3-Pad4) -> unconnected-(J3-Pad4)
- R1 pad 1: Net-(J2-Pad24) -> Net-(J3-Pad24)
- R2 pad 1: Net-(J3-Pad4) -> Net-(J3-Pad22)
- R2 pad 2: Net-(U3B-PIO2_28) -> Net-(U3B-PIO2_26)
- R3 pad 1: Net-(J3-Pad2) -> Net-(J3-Pad23)
- R3 pad 2: Net-(U3B-PIO2_26) -> Net-(U3B-PIO2_25)
- U2 pad 1: GND -> unconnected-(U2-GND/HEATSINK-Pad1)
- U2 pad 10: GND -> unconnected-(U2-GND/HEATSINK-Pad10)
- U2 pad 11: GND -> unconnected-(U2-GND/HEATSINK-Pad11)
- U2 pad 5: unconnected-(U2-*EN-Pad5) -> GND
- U2 pad 6: unconnected-(U2-PG/*RESET-Pad6) -> Net-(U2-PG/*RESET)
- U2 pad 7: unconnected-(U2-FB/SENSE-Pad7) -> /Alimentacion/V18
- U3 pad A15: unconnected-(U3B-PMIC_IRQ_N-PadA15) -> Net-(U3B-PMIC_IRQ_N)
- U3 pad A16: unconnected-(U3B-LDO_ENABLE-PadA16) -> GND
- U3 pad B14: unconnected-(U3B-XTALIN-PadB14) -> GND
- U3 pad B15: unconnected-(U3B-RESETN-PadB15) -> Net-(U3B-RESETN)
- U3 pad B17: unconnected-(U3B-RTCXIN-PadB17) -> GND
- U3 pad C2: unconnected-(U3B-VREFN-PadC2) -> GND
- U3 pad C4: unconnected-(U3B-VDDA_BIAS-PadC4) -> /Alimentacion/V18
- U3 pad C5: unconnected-(U3B-VDDCORE-PadC5) -> /Alimentacion/V18
- U3 pad D2: unconnected-(U3B-VREFP-PadD2) -> /Alimentacion/V18
- U3 pad D9: unconnected-(U3B-VDDCORE-PadD9) -> /Alimentacion/V18
- U3 pad F14: unconnected-(U3B-VDDCORE-PadF14) -> /Alimentacion/V18
- U3 pad J14: unconnected-(U3B-VDDCORE-PadJ14) -> /Alimentacion/V18
- U3 pad J4: unconnected-(U3B-VDDCORE-PadJ4) -> /Alimentacion/V18
- U3 pad L17: unconnected-(U3B-PIO2_25-PadL17) -> Net-(U3B-PIO2_25)
- U3 pad N15: Net-(U3B-PIO2_28) -> unconnected-(U3B-PIO2_28-PadN15)
- U3 pad P9: unconnected-(U3B-VDDCORE-PadP9) -> /Alimentacion/V18
- U3 pad R14: unconnected-(U3B-VDDCORE-PadR14) -> /Alimentacion/V18
- U3 pad R5: unconnected-(U3B-VDDCORE-PadR5) -> /Alimentacion/V18
Routing:
- net /Alimentacion/V18: track 0.00 -> 21.6 mm
- net GND: track 0.00 -> 20.4 mm, vias 0 -> 1
